File: Caps32Project.kicad_pcb (KiCad board)
At the start: 2 copper layers, 22.5 x 25.5 mm, 37 parts, among them J1 Sh 1.0, J2 Sh 1.0, J3 USB_C_Receptacle_PowerOnly_6P, Q1 AO3401A, Q2 MBT3904DW1, SW1 Boot, SW2 Reset, U1 AP2112K-3.3, U2 ESP32-WROOM-32U, U3 MCP73831-2-OT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

Commit message: Update Board
Parts:
- removed Bat+1, Bat-1: TestPoint, TestPoint:TestPoint_Pad_D1.5mm
- removed D3: LED, LED_SMD:LED_0402_1005Metric
- removed U5: MAX17048G_T10, Custom:SON50P200X200X80-9N
- added C10: 10uF, Capacitor_SMD:C_0402_1005Metric, B.Cu at (128.8, 44.3)
- added C11: 10uF, Capacitor_SMD:C_0402_1005Metric, B.Cu at (124.3, 41.8)
- added R10: 5.1K, Resistor_SMD:R_0402_1005Metric, B.Cu at (137.7, 44.6)
- added R11: 442K, Resistor_SMD:R_0805_2012Metric, B.Cu at (124.0, 50.3)
- added R12: 160K, Resistor_SMD:R_0805_2012Metric, B.Cu at (124.1, 54.0)
- added R13: 5.1K, Resistor_SMD:R_0402_1005Metric, B.Cu at (126.2, 44.0)
- added TP1: BAT+, TestPoint:TestPoint_Pad_D1.5mm, B.Cu at (142.7, 43.6)
- added TP2: BAT-, TestPoint:TestPoint_Pad_D1.5mm, B.Cu at (142.6, 40.7)
- C1, C2, C3, C7, C9: value 1.0uF -> 10uF; footprint Capacitor_SMD:C_0201_0603Metric -> Capacitor_SMD:C_0402_1005Metric; moved to B.Cu
- C4, C5: value 4.7uF -> 10uF; moved to B.Cu
- C6, C8, D2, D4, J3, Q1, Q2, R2, R3, R4, R5, U1, U3, U4: moved to B.Cu
- D1: value SS34 -> SS54; moved to B.Cu
- J1, J2: footprint Connector_JST:JST_SH_SM04B-SRSS-TB_1x04-1MP_P1.00mm_Horizontal -> Connector_JST:JST_SH_BM04B-SRSS-TB_1x04-1MP_P1.00mm_Vertical; moved to B.Cu
- R1: value 10K -> 100K; moved to B.Cu
- R6, R7: value 1K -> 5.1K; footprint Resistor_SMD:R_0201_0603Metric -> Resistor_SMD:R_0402_1005Metric; moved to B.Cu
- R8: value 1K -> 5.1k; footprint Resistor_SMD:R_0201_0603Metric -> Resistor_SMD:R_0402_1005Metric; moved to B.Cu
- R9: value 2K -> 5.1K; moved to B.Cu
- SW1: value Boot -> Reset; footprint Button_Switch_SMD:SW_SPST_CK_KMS2xxGP -> Button_Switch_SMD:SW_Push_SPST_NO_Alps_SKRK
- SW2: value Reset -> Boot; footprint Button_Switch_SMD:SW_SPST_CK_KMS2xxGP -> Button_Switch_SMD:SW_Push_SPST_NO_Alps_SKRK
- U2: moved to F.Cu
- moved SW1 60.3 mm to (142.8, 41.7), turned to 90 degrees
- moved D5 55.7 mm to (142.9, 52.5)
- moved J2 54.3 mm to (137.1, 40.7), turned to 180 degrees
- moved J3 50.9 mm to (141.6, 51.8), turned to -90 degrees
- moved C8 49.3 mm to (134.4, 44.9), turned to 0 degrees
- moved U1 47.6 mm to (135.2, 56.2)
- moved U4 47.5 mm to (134.6, 47.9), turned to 180 degrees
- moved C2 47.5 mm to (132.0, 44.3)
- moved Q1 45.3 mm to (135.5, 52.6)
- moved J1 45.1 mm to (129.2, 40.7), turned to 180 degrees
- moved C5 45.0 mm to (132.9, 53.5), turned to -90 degrees
- moved R4 44.4 mm to (131.5, 56.3), turned to 90 degrees
- moved C1 44.2 mm to (132.6, 56.9)
- moved SW2 43.0 mm to (142.8, 47.4), turned to -90 degrees
- moved C3 42.7 mm to (133.1, 44.3), turned to -90 degrees
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Connections:
- C4 pad 1: VBUS -> +3V3
- C9 pad 1: +BATT -> +3V3
- Q2 pad 6: CHIP_PU -> EN
- R5 pad 2: CHIP_PU -> EN
- R7 pad 2: Net-(D3-A) -> SCL
- SW1 pad 1: CHIP_PU -> GND
- SW1 pad 2: GND -> EN
- SW2 pad 1: 0 -> GND
- SW2 pad 2: GND -> 0
- U2 pad 14: unconnected-(U2-IO12-Pad14) -> SENSE
- U2 pad 3: CHIP_PU -> EN
Routing:
- net GND: track 116.3 -> 61.8 mm, vias 18 -> 9
- net CHIP_PU: track 42.8 -> 0.00 mm, vias 4 -> 0
- net EN: track 0.00 -> 28.4 mm, vias 0 -> 2
- net LED: track 17.6 -> 0.98 mm
- net +3V3: track 67.2 -> 51.8 mm, vias 8 -> 7
- net SDA: track 21.2 -> 7.97 mm, vias 2 -> 1
- net VBUS: track 21.2 -> 32.4 mm, vias 2 -> 3
- net SCL: track 18.2 -> 7.94 mm, vias 4 -> 1
- net Net-(D2-K): track 4.58 -> 11.2 mm, vias 0 -> 2
- net SENSE: track 0.00 -> 6.17 mm, vias 0 -> 1
- net RTS: track 12.7 -> 8.29 mm, vias 0 -> 2
- net TX: track 6.01 -> 10.4 mm
- net RGB_DI: track 4.98 -> 9.00 mm, vias 1 -> 0
- net 0: track 28.1 -> 32.0 mm, vias 2 -> 1
- net RX: track 8.78 -> 12.5 mm
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- added copper zone on B.Cu, net GND
Other:
- board size 22.5 x 25.5 mm -> 23.9 x 20.7 mm

Commit message: Update Board
Parts:
- added SW3: SW_SPDT, Button_Switch_SMD:SW_SPDT_PCM12, F.Cu at (64.4, 82.3)
- C8: footprint Capacitor_SMD:C_0201_0603Metric -> Capacitor_SMD:C_0402_1005Metric
- D2, D4: moved to F.Cu
- J1, J2: value Sh 1.0 -> SH1.0
- R1, R2, R3, R4, R5: footprint Resistor_SMD:R_0201_0603Metric -> Resistor_SMD:R_0402_1005Metric
- moved SW1 100.1 mm to (51.0, 81.5)
- moved D5 93.1 mm to (54.5, 81.5), turned to 90 degrees
- moved SW2 91.5 mm to (57.9, 81.5), turned to 90 degrees
- moved J3 90.7 mm to (55.9, 81.2), turned to 180 degrees
- moved C8 85.6 mm to (51.0, 64.3)
- moved C3 85.3 mm to (54.0, 76.2), turned to 0 degrees
- moved TP2 84.4 mm to (65.9, 75.9), turned to -90 degrees
- moved U4 82.9 mm to (52.8, 61.1), turned to -90 degrees
- moved TP1 82.3 mm to (65.9, 73.3), turned to -90 degrees
- moved C2 82.2 mm to (54.2, 70.9), turned to 0 degrees
- moved U1 82.1 mm to (55.0, 73.6), turned to -90 degrees
- moved J2 80.2 mm to (59.5, 61.1)
- moved R10 79.5 mm to (60.6, 64.3)
- moved D1 78.8 mm to (51.0, 73.3), turned to -90 degrees
- moved R7 77.7 mm to (60.9, 65.4), turned to 180 degrees
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Connections:
- C2 pad 1: +3V3 -> Net-(SW3-A)
- C3 pad 1: +3V3 -> Net-(SW3-A)
- J1 pad 1: TX -> DTR
- J1 pad 2: RX -> RTS
- J1 pad 3: DTR -> TX
- J1 pad 4: RTS -> RX
- J1 pad MP: (no net) -> GND
- J2 pad 2: SDA -> SCL
- J2 pad 3: SCL -> SDA
- J2 pad MP: (no net) -> GND
- R10 pad 2: SDA -> SCL
- R7 pad 2: SCL -> SDA
- U1 pad 5: +3V3 -> Net-(SW3-A)
Routing:
- net GND: track 61.8 -> 25.8 mm, vias 9 -> 24
- net Net-(SW3-A): track 0.00 -> 21.6 mm, vias 0 -> 3
- net SCL: track 7.94 -> 26.2 mm, vias 1 -> 2
- net SDA: track 7.97 -> 25.1 mm, vias 1 -> 4
- net +BATT: track 27.5 -> 15.4 mm, vias 2 -> 0
- net LED: track 0.98 -> 13.0 mm
- net 0: track 32.0 -> 20.4 mm, vias 1 -> 2
- net EN: track 28.4 -> 39.9 mm, vias 2 -> 4
- net RX: track 12.5 -> 3.15 mm
- net +3V3: track 51.8 -> 59.1 mm, vias 7 -> 5
- net TX: track 10.4 -> 3.26 mm
- net SENSE: track 6.17 -> 11.9 mm
- net RGB_DI: track 9.00 -> 13.9 mm, vias 0 -> 2
- net VBUS: track 32.4 -> 29.4 mm, vias 3 -> 4
- net Net-(U4-CPOUT): track 1.20 -> 3.23 mm
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- added copper zone on F.Cu, net GND
Other:
- board size 23.9 x 20.7 mm -> 19.9 x 26.3 mm

Commit message: Update Caps32Project.kicad_pcb
Routing:
- net GND: track 25.8 -> 32.7 mm
- net EN: track 39.9 -> 39.4 mm
Changed lines of the file:
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@@
 		(tags "LED")
 		(property "Reference" "D4"
-			(at 0 -1.17 360)
+			(at 0 -1.17 0)
 			(layer "F.SilkS")
 			(hide yes)
@@
 		)
 		(property "Value" "LED"
-			(at 0 1.17 360)
+			(at 0 1.17 0)
 			(layer "F.Fab")
 			(effects
@@
 		)
 		(fp_text user "${REFERENCE}"
-			(at 0 0 360)
+			(at 0 0 0)
 			(layer "F.Fab")
 			(effects
@@
 		(tags "capacitor")
 		(property "Reference" "C7"
-			(at 0 1.16 360)
+			(at 0 1.16 0)
 			(layer "B.SilkS")
 			(hide yes)
@@
 		)
 		(property "Value" "10uF"
-			(at 0 -1.16 360)
+			(at 0 -1.16 0)
 			(layer "B.Fab")
 			(effects
@@
 		)
 		(fp_text user "${REFERENCE}"
-			(at 0 0 360)
+			(at 0 0 0)
 			(layer "B.Fab")
 			(effects
@@
 		(tags "capacitor")
 		(property "Reference" "C11"
-			(at 0 1.16 360)
+			(at 0 1.16 0)
 			(layer "B.SilkS")
 			(hide yes)
@@
 		)
 		(property "Value" "10uF"
-			(at 0 -1.16 360)
+			(at 0 -1.16 0)
 			(layer "B.Fab")
 			(effects
@@
 		)
 		(fp_text user "${REFERENCE}"
-			(at 0 0 360)
+			(at 0 0 0)
 			(layer "B.Fab")
 			(effects
@@
 		(tags "capacitor")
 		(property "Reference" "C5"
-			(at 0 1.16 360)
+			(at 0 1.16 0)
 			(layer "B.SilkS")
 			(hide yes)
@@
 		)
 		(property "Value" "10uF"
-			(at 0 -1.16 360)
+			(at 0 -1.16 0)
 			(layer "B.Fab")
 			(effects
@@
 		)
 		(fp_text user "${REFERENCE}"
-			(at 0 0 360)
+			(at 0 0 0)
 			(layer "B.Fab")
 			(effects
@@
 		(tags "capacitor")
 		(property "Reference" "C8"
-			(at 0 1.16 360)
+			(at 0 1.16 0)
 			(layer "B.SilkS")
 			(hide yes)
@@
 		)
 		(property "Value" "0.1uF"
-			(at 0 -1.16 360)
+			(at 0 -1.16 0)
 			(layer "B.Fab")
 			(effects
@@
 		)
 		(fp_text user "${REFERENCE}"
-			(at 0 0 360)
+			(at 0 0 0)
 			(layer "B.Fab")
 			(effects
@@
 		)
 		(property "Value" "MBT3904DW1"
-			(at 0 -2 360)
+			(at 0 -2 0)
 			(layer "B.Fab")
 			(effects
@@
 		(tags "capacitor")
 		(property "Reference" "C2"
-			(at 0 1.16 360)
+			(at 0 1.16 0)
 			(layer "B.SilkS")
 			(hide yes)
@@
 		)
 		(property "Value" "10uF"
-			(at 0 -1.16 360)
+			(at 0 -1.16 0)
 			(layer "B.Fab")
 			(effects
@@
 		)
 		(fp_text user "${REFERENCE}"
-			(at 0 0 360)
+			(at 0 0 0)
 			(layer "B.Fab")
 			(effects
@@
 		(tags "resistor")
 		(property "Reference" "R12"
-			(at 0 1.65 360)
+			(at 0 1.65 0)
 			(layer "B.SilkS")
 			(hide yes)
@@
 		)
 		(property "Value" "160K"
-			(at 0 -1.65 360)
+			(at 0 -1.65 0)
 			(layer "B.Fab")
 			(effects
@@
 		)
 		(fp_text user "${REFERENCE}"
-			(at 0 0 360)
+			(at 0 0 0)
 			(layer "B.Fab")
 			(effects
@@
 		(tags "connector JST SH vertical")
 		(property "Reference" "J2"
-			(at 0 3.3 360)
+			(at 0 3.3 0)
 			(layer "B.SilkS")
 			(hide yes)
@@
 		)
 		(property "Value" "SH1.0"
-			(at 0 -3.3 360)
+			(at 0 -3.3 0)
 			(layer "B.Fab")
 			(effects
@@
 		)
 		(fp_text user "${REFERENCE}"
-			(at 0 0.25 360)
+			(at 0 0.25 0)
 			(layer "B.Fab")
 			(effects
@@
 		(tags "capacitor")
 		(property "Reference" "C1"
-			(at 0 1.16 360)
+			(at 0 1.16 0)
 			(layer "B.SilkS")
 			(hide yes)
@@
 		)
 		(property "Value" "10uF"
-			(at 0 -1.16 360)
+			(at 0 -1.16 0)
 			(layer "B.Fab")
 			(effects
@@
 		)
 		(fp_text user "${REFERENCE}"
-			(at 0 0 360)
+			(at 0 0 0)
 			(layer "B.Fab")
 			(effects
@@
 		(tags "resistor")
 		(property "Reference" "R8"
-			(at 0 1.17 360)
+			(at 0 1.17 0)
 			(layer "B.SilkS")
 			(hide yes)
@@
 		)
 		(property "Value" "5.1k"
-			(at 0 -1.17 360)
+			(at 0 -1.17 0)
 			(layer "B.Fab")
 			(effects
@@
 		)
 		(fp_text user "${REFERENCE}"
-			(at 0 0 360)
+			(at 0 0 0)
 			(layer "B.Fab")
 			(effects
@@
 		(tags "capacitor")
 		(property "Reference" "C9"
-			(at 0 1.16 360)
+			(at 0 1.16 0)
 			(layer "B.SilkS")
 			(hide yes)
@@
 		)
 		(property "Value" "10uF"
-			(at 0 -1.16 360)
+			(at 0 -1.16 0)
 			(layer "B.Fab")
 			(effects
@@
 		)
 		(fp_text user "${REFERENCE}"
-			(at 0 0 360)
+			(at 0 0 0)
 			(layer "B.Fab")
 			(effects
@@
 		(tags "capacitor")
 		(property "Reference" "C3"
-			(at 0 1.16 360)
+			(at 0 1.16 0)
 			(layer "B.SilkS")
 			(hide yes)
@@
 		)
 		(property "Value" "10uF"
-			(at 0 -1.16 360)
+			(at 0 -1.16 0)
 			(layer "B.Fab")
 			(effects
@@
 		)
 		(fp_text user "${REFERENCE}"
-			(at 0 0 360)
+			(at 0 0 0)
 			(layer "B.Fab")
 			(effects
@@
 	)
 	(segment
+		(start 50.748527 60.035)
+		(end 51.298529 59.484998)
+		(width 0.2)
+		(layer "F.Cu")
+		(net 2)
+	)
+	(segment
+		(start 50.3 60.035)
+		(end 50.748527 60.035)
+		(width 0.2)
+		(layer "F.Cu")
+		(net 2)
+	)
+	(segment
+		(start 56.309998 59.484998)
+		(end 56.75 59.925)
+		(width 0.2)
+		(layer "F.Cu")
+		(net 2)
+	)
+	(segment
 		(start 65.85 75.95)
 		(end 65.85 78.9825)
@@
 	)
 	(segment
+		(start 51.298529 59.484998)
+		(end 56.309998 59.484998)
+		(width 0.2)
+		(layer "F.Cu")
+		(net 2)
+	)
+	(segment
 		(start 65.85 78.9825)
 		(end 65.5825 79.25)
@@
 	)
 	(segment
-		(start 56.855 61.305)
-		(end 50.3 61.305)
+		(start 51.820686 63)
+		(end 51.35 62.529314)
 		(width 0.2)
 		(layer "F.Cu")
@@
 	)
 	(segment
+		(start 51.35 61.525)
+		(end 51.13 61.305)
+		(width 0.2)
+		(layer "F.Cu")
+		(net 4)
+	)
+	(segment
 		(start 52.875 78.9)
 		(end 52.275 78.3)
@@
 	)
 	(segment
-		(start 57.175 61.625)
-		(end 56.855 61.305)
+		(start 51.35 62.529314)
+		(end 51.35 61.525)
 		(width 0.2)
 		(layer "F.Cu")
@@
 	)
 	(segment
+		(start 55.75 63)
+		(end 51.820686 63)
+		(width 0.2)
+		(layer "F.Cu")
+		(net 4)
+	)
+	(segment
 		(start 53.9 79.05)
 		(end 53.75 78.9)
@@
 	)
 	(segment
+		(start 51.13 61.305)
+		(end 50.3 61.305)
+		(width 0.2)
+		(layer "F.Cu")
+		(net 4)
+	)
+	(segment
 		(start 52.425 70.1125)
 		(end 53.585 68.9525)
@@
 	)
 	(segment
+		(start 54.35 63.4)
+		(end 51.655 63.4)
+		(width 0.2)
+		(layer "F.Cu")
+		(net 10)
+	)
+	(segment
 		(start 51.95 69.675)
 		(end 52.625 69)
@@
 	)
 	(segment
-		(start 54.4 62.575)
-		(end 50.3 62.575)
-		(width 0.2)
-		(layer "F.Cu")
-		(net 10)
-	)
-	(segment
-		(start 54.775 65.36)
-		(end 54.775 62.95)
+		(start 52.625 64.385)
+		(end 52.565 64.325)
 		(width 0.2)
 		(layer "F.Cu")
@@
 	)
 	(segment
-		(start 52.625 64.385)
-		(end 52.565 64.325)
+		(start 54.775 63.825)
+		(end 54.35 63.4)
 		(width 0.2)
 		(layer "F.Cu")
@@
 	)
 	(segment
-		(start 54.775 62.95)
-		(end 54.4 62.575)
+		(start 54.775 65.36)
+		(end 54.775 63.825)
 		(width 0.2)
 		(layer "F.Cu")
@@
 	)
 	(segment
+		(start 50.83 62.575)
+		(end 50.3 62.575)
+		(width 0.2)
+		(layer "F.Cu")
+		(net 10)
+	)
+	(segment
+		(start 51.655 63.4)
+		(end 50.83 62.575)
+		(width 0.2)
+		(layer "F.Cu")
+		(net 10)
+	)
+	(segment
 		(start 61.16 65.36)
 		(end 54.775 65.36)
@@
 			)
 		)
+	)
+	(zone
+		(net 0)
+		(net_name "")
+		(layers "F&B.Cu")
+		(hatch edge 0.5)
+		(connect_pads
+			(clearance 0)
+		)
+		(min_thickness 0.25)
+		(filled_areas_thickness no)
+		(keepout
+			(tracks not_allowed)
+			(vias not_allowed)
+			(pads not_allowed)
+			(copperpour not_allowed)
+			(footprints not_allowed)
+		)
+		(fill
+			(thermal_gap 0.5)
+			(thermal_bridge_width 0.5)
+		)
+		(polygon
+			(pts
+				(xy 51.475 59.725) (xy 51.475 62.475) (xy 54.125 62.475) (xy 54.125 59.725)
+			)
+		)

Commit message: Update Board
Parts:
- moved R7 0.86 mm to (60.0, 65.5)
- moved R10 0.34 mm to (60.9, 64.3), turned to 0 degrees
Connections:
- J2 pad 1: +3V3 -> SCL
- J2 pad 2: SCL -> SDA
- J2 pad 3: SDA -> +3V3
- R10 pad 2: SCL -> SDA
- R7 pad 2: SDA -> SCL
Routing:
- net GND: track 32.7 -> 38.8 mm, vias 24 -> 25
- net SCL: track 26.2 -> 27.9 mm, vias 2 -> 3
- net SDA: track 25.1 -> 24.1 mm

Commit message: Update Board
Parts:
- added G***: LOGO, LOGO, B.Cu at (67.0, 59.8)
- D2: moved to B.Cu
- moved C10 1.02 mm to (60.7, 67.2), turned to 90 degrees
- moved D2 1.01 mm to (63.1, 78.5), turned to -90 degrees
- moved C9 0.63 mm to (61.8, 65.9), turned to -90 degrees
- moved C4 0.62 mm to (63.0, 64.7)
Routing:
- net GND: track 38.8 -> 46.5 mm, vias 25 -> 20
- net +3V3: track 58.8 -> 63.6 mm, vias 5 -> 7
- net EN: track 39.4 -> 43.7 mm, vias 4 -> 3
- net VBUS: track 29.4 -> 32.2 mm
- net SENSE: track 11.9 -> 14.3 mm
- net Net-(D1-K): track 15.9 -> 17.9 mm
- net 0: track 20.4 -> 22.3 mm
- net Net-(SW3-A): track 21.6 -> 23.6 mm
- net Net-(D2-K): track 10.9 -> 8.93 mm, vias 3 -> 2
- net Net-(D4-A): track 0.00 -> 1.64 mm
- net Net-(D2-A): track 0.00 -> 1.25 mm, vias 1 -> 0
- net SCL: track 27.9 -> 28.7 mm
- net RGB_DI: track 13.9 -> 13.3 mm
- net SDA: track 24.1 -> 24.4 mm, vias 4 -> 3
Other:
- board text added: "+"
- board text added: "-"

Commit message: Update Board
Parts:
- moved G*** 0.75 mm to (66.2, 59.9)
