File: Caps32Project.kicad_sch (KiCad schematic)
At the start: 37 parts, among them J1 Ph 2.0, J2 Sh 1.0, J4 Sh 2.0, P1 USB_C_Plug_USB2.0, Q1 AO3401A, Q2 MBT3904DW1, SW1 Reset, SW2 Boot, U1 MPU-6050, U2 MAX17048G_T10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

Commit message: Update Board
Parts:
- removed D3: WS2812B, LED_SMD:LED_WS2812B_PLCC4_5.0x5.0mm_P3.2mm, symbol LED:WS2812B
- removed J1: Ph 2.0, Connector_JST:JST_PH_S2B-PH-SM4-TB_1x02-1MP_P2.00mm_Horizontal, symbol Connector_Generic:Conn_01x02
- removed P1: USB_C_Plug_USB2.0, Connector_USB:USB_C_Receptacle_XKB_U262-16XN-4BVC11, symbol Connector:USB_C_Plug_USB2.0
- removed TP4: +5V, TestPoint:TestPoint_Pad_D1.0mm, symbol Connector:TestPoint_Small
- removed U6: ESP32-WROOM-32D, RF_Module:ESP32-WROOM-32D, symbol RF_Module:ESP32-WROOM-32D
- added Bat+1, Bat-1: TestPoint, TestPoint:TestPoint_Pad_D1.5mm, symbol Connector:TestPoint
- added D5: WS2812B-2020, LED_SMD:LED_WS2812B-2020_PLCC4_2.0x2.0mm, symbol LED:WS2812B-2020
- added J3: USB_C_Receptacle_PowerOnly_6P, Connector_USB:USB_C_Receptacle_GCT_USB4135-GF-A_6P_TopMnt_Horizontal, symbol Connector:USB_C_Receptacle_PowerOnly_6P
- added U2: ESP32-WROOM-32U, RF_Module:ESP32-WROOM-32U, symbol RF_Module:ESP32-WROOM-32U
- C1: renamed from C13; footprint Capacitor_SMD:C_0402_1005Metric_Pad0.74x0.62mm_HandSolder -> Capacitor_SMD:C_0201_0603Metric
- C2: renamed from C7; footprint Capacitor_SMD:C_0402_1005Metric_Pad0.74x0.62mm_HandSolder -> Capacitor_SMD:C_0201_0603Metric
- C3: renamed from C8; footprint Capacitor_SMD:C_0402_1005Metric_Pad0.74x0.62mm_HandSolder -> Capacitor_SMD:C_0201_0603Metric
- C4: renamed from C2; footprint Capacitor_SMD:C_0402_1005Metric_Pad0.74x0.62mm_HandSolder -> Capacitor_SMD:C_0402_1005Metric
- C5: footprint Capacitor_SMD:C_0402_1005Metric_Pad0.74x0.62mm_HandSolder -> Capacitor_SMD:C_0402_1005Metric
- C6: renamed from C3; footprint Capacitor_SMD:C_0402_1005Metric_Pad0.74x0.62mm_HandSolder -> Capacitor_SMD:C_0603_1608Metric
- C7: renamed from C6; footprint Capacitor_SMD:C_0402_1005Metric_Pad0.74x0.62mm_HandSolder -> Capacitor_SMD:C_0201_0603Metric
- C8: renamed from C4; footprint Capacitor_SMD:C_0402_1005Metric_Pad0.74x0.62mm_HandSolder -> Capacitor_SMD:C_0201_0603Metric
- C9: renamed from C1; footprint Capacitor_SMD:C_0402_1005Metric_Pad0.74x0.62mm_HandSolder -> Capacitor_SMD:C_0201_0603Metric
- D2: footprint LED_SMD:LED_0402_1005Metric_Pad0.77x0.64mm_HandSolder -> LED_SMD:LED_0402_1005Metric
- D3: renamed from D1; footprint LED_SMD:LED_0402_1005Metric_Pad0.77x0.64mm_HandSolder -> LED_SMD:LED_0402_1005Metric
- D4: renamed from D5; footprint LED_SMD:LED_0402_1005Metric_Pad0.77x0.64mm_HandSolder -> LED_SMD:LED_0402_1005Metric
- J1: renamed from J4; value Sh 2.0 -> Sh 1.0
- R1: renamed from R5; footprint Resistor_SMD:R_0402_1005Metric_Pad0.72x0.64mm_HandSolder -> Resistor_SMD:R_0201_0603Metric
- R2: renamed from R7; footprint Resistor_SMD:R_0402_1005Metric_Pad0.72x0.64mm_HandSolder -> Resistor_SMD:R_0201_0603Metric
- R3: renamed from R8; footprint Resistor_SMD:R_0402_1005Metric_Pad0.72x0.64mm_HandSolder -> Resistor_SMD:R_0201_0603Metric
- R4: footprint Resistor_SMD:R_0402_1005Metric_Pad0.72x0.64mm_HandSolder -> Resistor_SMD:R_0201_0603Metric
- R5: renamed from R6; footprint Resistor_SMD:R_0402_1005Metric_Pad0.72x0.64mm_HandSolder -> Resistor_SMD:R_0201_0603Metric
- R6: renamed from R2; footprint Resistor_SMD:R_0402_1005Metric_Pad0.72x0.64mm_HandSolder -> Resistor_SMD:R_0201_0603Metric
- R7: renamed from R1; footprint Resistor_SMD:R_0402_1005Metric_Pad0.72x0.64mm_HandSolder -> Resistor_SMD:R_0201_0603Metric
- R8: renamed from R9; footprint Resistor_SMD:R_0402_1005Metric_Pad0.72x0.64mm_HandSolder -> Resistor_SMD:R_0201_0603Metric
- R9: renamed from R3; footprint Resistor_SMD:R_0402_1005Metric_Pad0.72x0.64mm_HandSolder -> Resistor_SMD:R_0402_1005Metric
- U4: renamed from U1; footprint Sensor_Motion:InvenSense_QFN-24_4x4mm_P0.5mm -> Sensor_Motion:InvenSense_QFN-24_4x4mm_P0.5mm_NoMask
- renumbered D4 to D1, SW2 to SW1, SW1 to SW2, U5 to U1, U4 to U3, U2 to U5
Connections:
- net +3V3: now also D5.4 (VDD), U2.2 (VDD)
- net +BATT: now also Bat+1.1
- net 0: now also U2.25 (IO0)
- net CHIP_PU: now also U2.3 (EN)
- net GND: now also Bat-1.1, D5.2 (VSS), J3.A12 (GND), J3.B12 (GND), U2.1 (GND), U2.15 (GND), U2.38 (GND), U2.39 (GND)
- net LED: now also U2.16 (IO13)
- net RGB_DI: now also D5.3 (DIN), U2.24 (IO2)
- net RX: now also U2.35 (TXD0/IO1)
- net SCL: now also U2.36 (IO22)
- net SDA: now also U2.37 (IO23)
- net TX: now also U2.34 (RXD0/IO3)
- net VBUS: now also J3.A9 (VBUS), J3.B9 (VBUS)
- no-connect marks 40 -> 38

Commit message: Update sch
Parts:
- removed Bat+1, Bat-1: TestPoint, TestPoint:TestPoint_Pad_D1.5mm, symbol Connector:TestPoint
- removed C9: 1.0uF, Capacitor_SMD:C_0201_0603Metric, symbol Device:C
- removed SW1: Boot, Button_Switch_SMD:SW_SPST_CK_KMS2xxGP, symbol Switch:CK_KMS2xxGP
- removed SW2: Reset, Button_Switch_SMD:SW_SPST_CK_KMS2xxGP, symbol Switch:CK_KMS2xxGP
- removed U5: MAX17048G_T10, Custom:SON50P200X200X80-9N, symbol Custom:MAX17048G_T10
- added J4: Ph 2.0, Connector_JST:JST_PH_S2B-PH-SM4-TB_1x02-1MP_P2.00mm_Horizontal, symbol Connector_Generic:Conn_01x02
- added SW1: Reset, symbol Switch:SW_Push
- added SW2: Boot, symbol Switch:SW_Push
- J1, J2: footprint Connector_JST:JST_SH_SM04B-SRSS-TB_1x04-1MP_P1.00mm_Horizontal -> Connector_JST:JST_SH_BM04B-SRSS-TB_1x04-1MP_P1.00mm_Vertical
Connections:
- net +BATT: now also J4.1 (Pin_1)
- net 0: now also SW2.2
- net CHIP_PU: no longer R5.2, U2.3 (EN)
- net GND: now also J4.2 (Pin_2), SW1.1, SW2.1
- new net EN: R5.2, SW1.2, U2.3 (EN)
- no-connect marks 38 -> 35
Other:
- moved on the sheet: C7, D5, R7, R8

Commit message: Update Board
Parts:
- removed D3: LED, LED_SMD:LED_0402_1005Metric, symbol Device:LED
- removed J4: Ph 2.0, Connector_JST:JST_PH_S2B-PH-SM4-TB_1x02-1MP_P2.00mm_Horizontal, symbol Connector_Generic:Conn_01x02
- added C10, C11, C9: 10uF, Capacitor_SMD:C_0402_1005Metric, symbol Device:C
- added R10, R13: 5.1K, Resistor_SMD:R_0402_1005Metric, symbol Device:R
- added R11: 442K, Resistor_SMD:R_0805_2012Metric, symbol Device:R
- added R12: 160K, Resistor_SMD:R_0805_2012Metric, symbol Device:R
- added TP1: BAT+, TestPoint:TestPoint_Pad_D1.5mm, symbol Connector:TestPoint
- added TP2: BAT-, TestPoint:TestPoint_Pad_D1.5mm, symbol Connector:TestPoint
- C1, C2, C3, C7: value 1.0uF -> 10uF; footprint Capacitor_SMD:C_0201_0603Metric -> Capacitor_SMD:C_0402_1005Metric
- C4, C5: value 4.7uF -> 10uF
- D1: value SS34 -> SS54
- R1: value 10K -> 100K
- R6, R7: value 1K -> 5.1K; footprint Resistor_SMD:R_0201_0603Metric -> Resistor_SMD:R_0402_1005Metric
- R8: value 1K -> 5.1k; footprint Resistor_SMD:R_0201_0603Metric -> Resistor_SMD:R_0402_1005Metric
- R9: value 2K -> 5.1K
- SW1, SW2: footprint (none) -> Button_Switch_SMD:SW_Push_SPST_NO_Alps_SKRK
Connections:
- net CHIP_PU is gone; now on net EN: Q2.6 (C1)
- net +3V3: now also C4.1, C10.1, C9.1, R10.1, R13.1
- net +BATT: now also R11.1, TP1.1
- net EN: now also C11.1, R13.2
- net GND: now also C10.2, C11.2, C9.2, R12.2, TP2.1
- net SCL: now also R7.2
- net SDA: now also R10.2
- net VBUS: no longer C4.1
- net SENSE: now reaches U2.14 (IO12)
- net SENSE: now also R11.2, R12.1
- no-connect marks 35 -> 34
Other:
- moved on the sheet: C7, D5, J2, R8, SW1, SW2

Commit message: Update Board
Parts:
- removed J1, J2: Sh 1.0, Connector_JST:JST_SH_BM04B-SRSS-TB_1x04-1MP_P1.00mm_Vertical, symbol Connector_Generic:Conn_01x04
- added J1, J2: SH1.0, Connector_JST:JST_SH_BM04B-SRSS-TB_1x04-1MP_P1.00mm_Vertical, symbol Connector_Generic_MountingPin:Conn_01x04_MountingPin
- added SW3: SW_SPDT, Button_Switch_SMD:SW_SPDT_PCM12, symbol Switch:SW_SPDT
- C8: footprint Capacitor_SMD:C_0201_0603Metric -> Capacitor_SMD:C_0402_1005Metric
- R1, R2, R3, R4, R5: footprint Resistor_SMD:R_0201_0603Metric -> Resistor_SMD:R_0402_1005Metric
Connections:
- net +3V3: now also J2.1 (Pin_1), SW3.2 (B); no longer C2.1, C3.1, U1.5 (VOUT)
- net DTR: now also J1.1 (Pin_1)
- net GND: now also J1.MP (MountPin), J2.4 (Pin_4), J2.MP (MountPin)
- net RTS: now also J1.2 (Pin_2)
- net RX: now also J1.4 (Pin_4)
- net SCL: now also R10.2, J2.2 (Pin_2); no longer R7.2
- net SDA: now also R7.2, J2.3 (Pin_3); no longer R10.2
- net TX: now also J1.3 (Pin_3)
- new net: C2.1, C3.1, SW3.1 (A), U1.5 (VOUT)
- no-connect marks 34 -> 35

Commit message: Update Board
Connections:
- net +3V3: now also J2.3 (Pin_3); no longer J2.1 (Pin_1)
- net SCL: now also J2.1 (Pin_1), R7.2; no longer J2.2 (Pin_2), R10.2
- net SDA: now also J2.2 (Pin_2), R10.2; no longer J2.3 (Pin_3), R7.2
Other:
- moved on the sheet: R7
Changed lines of the file:
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@@
 	(paper "A4")
 	(junction
-		(at 49.53 69.85)
+		(at 64.77 93.98)
 		(diameter 0)
 		(color 0 0 0 0)
 	)
 	(junction
-		(at 66.04 93.98)
+		(at 49.53 69.85)
 		(diameter 0)
 		(color 0 0 0 0)
@@
 	)
 	(junction
-		(at 57.15 104.14)
-		(diameter 0)
-		(color 0 0 0 0)
-	)
-	(junction
 		(at 74.93 135.89)
 		(diameter 0)
@@
 	)
 	(junction
+		(at 57.15 100.33)
+		(diameter 0)
+		(color 0 0 0 0)
+	)
+	(junction
 		(at 27.94 123.19)
 		(diameter 0)
@@
 	(wire
 		(pts
-			(xy 57.15 93.98) (xy 62.23 93.98)
+			(xy 57.15 92.71) (xy 62.23 92.71)
 		)
 		(stroke
@@
 	(wire
 		(pts
-			(xy 66.04 93.98) (xy 66.04 99.06)
-		)
-		(stroke
-			(width 0)
-			(type default)
-		)
-	)
-	(wire
-		(pts
 			(xy 199.39 134.62) (xy 199.39 138.43)
 		)
@@
 	(wire
 		(pts
-			(xy 66.04 104.14) (xy 57.15 104.14)
+			(xy 66.04 104.14) (xy 64.77 104.14)
 		)
 		(stroke
@@
 	(wire
 		(pts
-			(xy 57.15 104.14) (xy 53.34 104.14)
+			(xy 57.15 100.33) (xy 53.34 100.33)
 		)
 		(stroke
@@
 	(wire
 		(pts
-			(xy 53.34 104.14) (xy 53.34 100.33)
-		)
-		(stroke
-			(width 0)
-			(type default)
-		)
-	)
-	(wire
-		(pts
 			(xy 27.94 125.73) (xy 27.94 123.19)
 		)
@@
 	(wire
 		(pts
-			(xy 57.15 96.52) (xy 57.15 93.98)
+			(xy 49.53 69.85) (xy 49.53 77.47)
 		)
 		(stroke
@@
 	(wire
 		(pts
-			(xy 49.53 69.85) (xy 49.53 77.47)
+			(xy 59.69 99.06) (xy 59.69 100.33)
 		)
 		(stroke
@@
 	(wire
 		(pts
+			(xy 62.23 92.71) (xy 62.23 93.98)
+		)
+		(stroke
+			(width 0)
+			(type default)
+		)
+	)
+	(wire
+		(pts
 			(xy 176.53 118.11) (xy 176.53 124.46)
 		)
@@
 	(wire
 		(pts
+			(xy 64.77 93.98) (xy 64.77 104.14)
+		)
+		(stroke
+			(width 0)
+			(type default)
+		)
+	)
+	(wire
+		(pts
 			(xy 130.81 120.65) (xy 137.16 120.65)
 		)
@@
 	(wire
 		(pts
+			(xy 59.69 100.33) (xy 57.15 100.33)
+		)
+		(stroke
+			(width 0)
+			(type default)
+		)
+	)
+	(wire
+		(pts
 			(xy 191.77 118.11) (xy 191.77 124.46)
 		)
@@
 	(wire
 		(pts
+			(xy 66.04 99.06) (xy 59.69 99.06)
+		)
+		(stroke
+			(width 0)
+			(type default)
+		)
+	)
+	(wire
+		(pts
 			(xy 130.81 118.11) (xy 130.81 120.65)
 		)
@@
 	(wire
 		(pts
-			(xy 62.23 93.98) (xy 66.04 93.98)
+			(xy 62.23 93.98) (xy 64.77 93.98)
 		)
 		(stroke
@@
 	(global_label "SDA"
 		(shape input)
-		(at 53.34 100.33 180)
+		(at 53.34 97.79 180)
 		(fields_autoplaced yes)
 		(effects
@@
 		)
 		(property "Intersheetrefs" "${INTERSHEET_REFS}"
-			(at 46.7867 100.33 0)
+			(at 46.7867 97.79 0)
 			(effects
 				(font
@@
 	(global_label "SCL"
 		(shape input)
-		(at 53.34 97.79 180)
+		(at 53.34 100.33 180)
 		(fields_autoplaced yes)
 		(effects
@@
 		)
 		(property "Intersheetrefs" "${INTERSHEET_REFS}"
-			(at 46.8472 97.79 0)
+			(at 46.8472 100.33 0)
 			(effects
 				(font
@@
 	(symbol
 		(lib_id "Device:R")
-		(at 57.15 100.33 0)
+		(at 57.15 96.52 0)
 		(unit 1)
 		(exclude_from_sim no)
@@
 		(dnp no)
 		(property "Reference" "R7"
-			(at 59.182 101.6 90)
+			(at 59.182 97.79 90)
 			(effects
 				(font
@@
 		)
 		(property "Value" "5.1K"
-			(at 57.15 102.362 90)
+			(at 57.15 98.552 90)
 			(effects
 				(font
@@
 		)
 		(property "Footprint" "Resistor_SMD:R_0402_1005Metric"
-			(at 55.372 100.33 90)
+			(at 55.372 96.52 90)
 			(effects
 				(font
@@
 		)
 		(property "Datasheet" "~"
-			(at 57.15 100.33 0)
+			(at 57.15 96.52 0)
 			(effects
 				(font
@@
 		)
 		(property "Description" "Resistor"
-			(at 57.15 100.33 0)
+			(at 57.15 96.52 0)
 			(effects
 				(font
@@
 	(symbol
 		(lib_id "power:+3V3")
-		(at 66.04 93.98 0)
-		(mirror y)
+		(at 64.77 93.98 0)
 		(unit 1)
 		(exclude_from_sim no)
@@
 		(dnp no)
 		(property "Reference" "#PWR07"
-			(at 66.04 97.79 0)
+			(at 64.77 97.79 0)
 			(effects
 				(font
@@
 		)
 		(property "Value" "+3V3"
-			(at 63.5 89.916 0)
+			(at 67.31 89.916 0)
 			(effects
 				(font
@@
 		)
 		(property "Footprint" ""
-			(at 66.04 93.98 0)
+			(at 64.77 93.98 0)
 			(effects
 				(font
@@
 		)
 		(property "Datasheet" ""
-			(at 66.04 93.98 0)
+			(at 64.77 93.98 0)
 			(effects
 				(font
@@
 		)
 		(property "Description" "Power symbol creates a global label with name \"+3V3\""
-			(at 66.04 93.98 0)
+			(at 64.77 93.98 0)
 			(effects
 				(font

Commit message: Update Board
Other:
- moved on the sheet: D5, R11, R12
Changed lines of the file:
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@@
 	)
 	(no_connect
-		(at 135.89 86.36)
+		(at 110.49 100.33)
 	)
 	(no_connect
@@
 	(wire
 		(pts
-			(xy 143.51 76.2) (xy 143.51 78.74)
+			(xy 118.11 90.17) (xy 118.11 92.71)
 		)
 		(stroke
@@
 	(wire
 		(pts
-			(xy 168.91 83.82) (xy 168.91 88.9)
+			(xy 143.51 97.79) (xy 143.51 102.87)
 		)
 		(stroke
@@
 	(wire
 		(pts
-			(xy 143.51 93.98) (xy 143.51 96.52)
+			(xy 118.11 107.95) (xy 118.11 110.49)
 		)
 		(stroke
@@
 	(global_label "RGB_DI"
 		(shape input)
-		(at 151.13 86.36 0)
+		(at 125.73 100.33 0)
 		(fields_autoplaced yes)
 		(effects
@@
 		)
 		(property "Intersheetrefs" "${INTERSHEET_REFS}"
-			(at 160.7676 86.36 0)
+			(at 135.3676 100.33 0)
 			(effects
 				(font
@@
 	(global_label "SENSE"
 		(shape input)
-		(at 168.91 86.36 0)
+		(at 143.51 100.33 0)
 		(fields_autoplaced yes)
 		(effects
@@
 		)
 		(property "Intersheetrefs" "${INTERSHEET_REFS}"
-			(at 177.9427 86.36 0)
+			(at 152.5427 100.33 0)
 			(effects
 				(font
@@
 	(symbol
 		(lib_id "power:+BATT")
-		(at 168.91 76.2 0)
+		(at 143.51 90.17 0)
 		(unit 1)
 		(exclude_from_sim no)
@@
 		(fields_autoplaced yes)
 		(property "Reference" "#PWR035"
-			(at 168.91 80.01 0)
+			(at 143.51 93.98 0)
 			(effects
 				(font
@@
 		)
 		(property "Value" "+BATT"
-			(at 168.91 71.12 0)
+			(at 143.51 85.09 0)
 			(effects
 				(font
@@
 		)
 		(property "Footprint" ""
-			(at 168.91 76.2 0)
+			(at 143.51 90.17 0)
 			(effects
 				(font
@@
 		)
 		(property "Datasheet" ""
-			(at 168.91 76.2 0)
+			(at 143.51 90.17 0)
 			(effects
 				(font
@@
 		)
 		(property "Description" "Power symbol creates a global label with name \"+BATT\""
-			(at 168.91 76.2 0)
+			(at 143.51 90.17 0)
 			(effects
 				(font
@@
 	(symbol
 		(lib_id "power:GND")
-		(at 168.91 96.52 0)
+		(at 143.51 110.49 0)
 		(unit 1)
 		(exclude_from_sim no)
@@
 		(fields_autoplaced yes)
 		(property "Reference" "#PWR038"
-			(at 168.91 102.87 0)
+			(at 143.51 116.84 0)
 			(effects
 				(font
@@
 		)
 		(property "Value" "GND"
-			(at 168.91 101.6 0)
+			(at 143.51 115.57 0)
 			(effects
 				(font
@@
 		)
 		(property "Footprint" ""
-			(at 168.91 96.52 0)
+			(at 143.51 110.49 0)
 			(effects
 				(font
@@
 		)
 		(property "Datasheet" ""
-			(at 168.91 96.52 0)
+			(at 143.51 110.49 0)
 			(effects
 				(font
@@
 		)
 		(property "Description" "Power symbol creates a global label with name \"GND\" , ground"
-			(at 168.91 96.52 0)
+			(at 143.51 110.49 0)
 			(effects
 				(font
@@
 	(symbol
 		(lib_id "power:GND")
-		(at 143.51 96.52 0)
+		(at 118.11 110.49 0)
 		(mirror y)
 		(unit 1)
@@
 		(fields_autoplaced yes)
 		(property "Reference" "#PWR037"
-			(at 143.51 102.87 0)
+			(at 118.11 116.84 0)
 			(effects
 				(font
@@
 		)
 		(property "Value" "GND"
-			(at 143.51 101.6 0)
+			(at 118.11 115.57 0)
 			(effects
 				(font
@@
 		)
 		(property "Footprint" ""
-			(at 143.51 96.52 0)
+			(at 118.11 110.49 0)
 			(effects
 				(font
@@
 		)
 		(property "Datasheet" ""
-			(at 143.51 96.52 0)
+			(at 118.11 110.49 0)
 			(effects
 				(font
@@
 		)
 		(property "Description" "Power symbol creates a global label with name \"GND\" , ground"
-			(at 143.51 96.52 0)
+			(at 118.11 110.49 0)
 			(effects
 				(font
@@
 	(symbol
 		(lib_id "Device:R")
-		(at 168.91 92.71 0)
+		(at 143.51 106.68 0)
 		(unit 1)
 		(exclude_from_sim no)
@@
 		(dnp no)
 		(property "Reference" "R12"
-			(at 170.942 93.98 90)
+			(at 145.542 107.95 90)
 			(effects
 				(font
@@
 		)
 		(property "Value" "160K"
-			(at 168.91 95.504 90)
+			(at 143.51 109.474 90)
 			(effects
 				(font
@@
 		)
 		(property "Footprint" "Resistor_SMD:R_0805_2012Metric"
-			(at 167.132 92.71 90)
+			(at 141.732 106.68 90)
 			(effects
 				(font
@@
 		)
 		(property "Datasheet" "~"
-			(at 168.91 92.71 0)
+			(at 143.51 106.68 0)
 			(effects
 				(font
@@
 		)
 		(property "Description" "Resistor"
-			(at 168.91 92.71 0)
+			(at 143.51 106.68 0)
 			(effects
 				(font
@@
 	(symbol
 		(lib_id "Device:R")
-		(at 168.91 80.01 0)
+		(at 143.51 93.98 0)
 		(unit 1)
 		(exclude_from_sim no)
@@
 		(dnp no)
 		(property "Reference" "R11"
-			(at 170.942 81.28 90)
+			(at 145.542 95.25 90)
 			(effects
 				(font
@@
 		)
 		(property "Value" "442K"
-			(at 168.91 82.55 90)
+			(at 143.51 96.52 90)
 			(effects
 				(font
@@
 		)
 		(property "Footprint" "Resistor_SMD:R_0805_2012Metric"
-			(at 167.132 80.01 90)
+			(at 141.732 93.98 90)
 			(effects
 				(font
@@
 		)
 		(property "Datasheet" "~"
-			(at 168.91 80.01 0)
+			(at 143.51 93.98 0)
 			(effects
 				(font
@@
 		)
 		(property "Description" "Resistor"
-			(at 168.91 80.01 0)
+			(at 143.51 93.98 0)
 			(effects
 				(font
@@
 	(symbol
 		(lib_id "power:+3V3")
-		(at 143.51 76.2 0)
+		(at 118.11 90.17 0)
 		(unit 1)
 		(exclude_from_sim no)
@@
 		(fields_autoplaced yes)
 		(property "Reference" "#PWR036"
-			(at 143.51 80.01 0)
+			(at 118.11 93.98 0)
 			(effects
 				(font
@@
 		)
 		(property "Value" "+3V3"
-			(at 143.51 71.12 0)
+			(at 118.11 85.09 0)
 			(effects
 				(font
@@
 		)
 		(property "Footprint" ""
-			(at 143.51 76.2 0)
+			(at 118.11 90.17 0)
 			(effects
 				(font
@@
 		)
 		(property "Datasheet" ""
-			(at 143.51 76.2 0)
+			(at 118.11 90.17 0)
 			(effects
 				(font
@@
 		)
 		(property "Description" "Power symbol creates a global label with name \"+3V3\""
-			(at 143.51 76.2 0)
+			(at 118.11 90.17 0)
 			(effects
 				(font
@@
 	(symbol
 		(lib_id "LED:WS2812B-2020")
-		(at 143.51 86.36 0)
+		(at 118.11 100.33 0)
 		(mirror y)
 		(unit 1)
@@
 		(dnp no)
 		(property "Reference" "D5"
-			(at 157.48 80.0414 0)
+			(at 132.08 94.0114 0)
 			(effects
 				(font
@@
 		)
 		(property "Value" "WS2812B-2020"
-			(at 157.48 82.5814 0)
+			(at 132.08 96.5514 0)
 			(effects
 				(font
@@
 		)
 		(property "Footprint" "LED_SMD:LED_WS2812B-2020_PLCC4_2.0x2.0mm"
-			(at 142.24 93.98 0)
+			(at 116.84 107.95 0)
 			(effects
 				(font
@@
 		)
 		(property "Datasheet" "https://cdn-shop.adafruit.com/product-files/4684/4684_WS2812B-2020_V1.3_EN.pdf"
-			(at 140.97 95.885 0)
+			(at 115.57 109.855 0)
 			(effects
 				(font
@@
 		)
 		(property "Description" "RGB LED with integrated controller, 2.0 x 2.0 mm, 12 mA"
-			(at 143.51 86.36 0)
+			(at 118.11 100.33 0)
 			(effects
 				(font
