File: Caps32Project.kicad_sch (KiCad schematic)
At the start: 37 parts, among them J1 Ph 2.0, J2 Sh 1.0, J4 Sh 2.0, P1 USB_C_Plug_USB2.0, Q1 AO3401A, Q2 MBT3904DW1, SW1 Reset, SW2 Boot, U1 MPU-6050, U2 MAX17048G_T10, U4 MCP73831-2-OT, U5 AP2112K-3.3, U6 ESP32-WROOM-32D

Commit message: Update Board
Parts:
- removed C1: 1.0uF, Capacitor_SMD:C_0402_1005Metric_Pad0.74x0.62mm_HandSolder, symbol Device:C
- removed D3: WS2812B, LED_SMD:LED_WS2812B_PLCC4_5.0x5.0mm_P3.2mm, symbol LED:WS2812B
- removed D5: LED, LED_SMD:LED_0402_1005Metric_Pad0.77x0.64mm_HandSolder, symbol Device:LED
- removed J1: Ph 2.0, Connector_JST:JST_PH_S2B-PH-SM4-TB_1x02-1MP_P2.00mm_Horizontal, symbol Connector_Generic:Conn_01x02
- removed J4: Sh 2.0, Connector_JST:JST_SH_SM04B-SRSS-TB_1x04-1MP_P1.00mm_Horizontal, symbol Connector_Generic:Conn_01x04
- removed Q2: MBT3904DW1, Package_TO_SOT_SMD:SOT-363_SC-70-6, symbol Transistor_BJT:MBT3904DW1
- removed SW1: Reset, Button_Switch_SMD:SW_SPST_CK_KMS2xxGP, symbol Switch:CK_KMS2xxGP
- removed SW2: Boot, Button_Switch_SMD:SW_SPST_CK_KMS2xxGP, symbol Switch:CK_KMS2xxGP
- removed TP4: +5V, TestPoint:TestPoint_Pad_D1.0mm, symbol Connector:TestPoint_Small
- removed U1: MPU-6050, Sensor_Motion:InvenSense_QFN-24_4x4mm_P0.5mm, symbol Sensor_Motion:MPU-6050
- removed U2: MAX17048G_T10, Custom:SON50P200X200X80-9N, symbol Custom:MAX17048G_T10
- removed U4: MCP73831-2-OT, Package_TO_SOT_SMD:SOT-23-5, symbol Battery_Management:MCP73831-5-OT
- removed U6: ESP32-WROOM-32D, RF_Module:ESP32-WROOM-32D, symbol RF_Module:ESP32-WROOM-32D
- added C4: 0.1uF, Capacitor_SMD:C_0201_0603Metric, symbol Device:C
- added D3: WS2812B-2020, LED_SMD:LED_WS2812B-2020_PLCC4_2.0x2.0mm, symbol LED:WS2812B-2020
- added R11, R12, R13: 100K, Resistor_SMD:R_0201_0603Metric, symbol Device:R
- added R3: 442K, Resistor_SMD:R_0805_2012Metric, symbol Device:R
- added R4: 160K, Resistor_SMD:R_0805_2012Metric, symbol Device:R
- added R5: 2K, Resistor_SMD:R_0402_1005Metric, symbol Device:R
- added SW1: Boot, Button_Switch_SMD:SW_SPST_CK_KMS2xxGP, symbol Switch:SW_SPST
- added SW2: Reset, Button_Switch_SMD:SW_SPST_CK_KMS2xxGP, symbol Switch:SW_SPST
- added TP1, TP2: TestPoint, TestPoint:TestPoint_Pad_D1.5mm, symbol Connector:TestPoint
- added U1: TP4057, Package_TO_SOT_SMD:TSOT-23-6, symbol Battery_Management:TP4057
- added U2: MPU-6050, Sensor_Motion:InvenSense_QFN-24_4x4mm_P0.5mm_NoMask, symbol Sensor_Motion:MPU-6050
- added U3: ESP32-C3-MINI-1, PCM_Espressif:ESP32-C3-MINI-1, symbol PCM_Espressif:ESP32-C3-MINI-1
- C1: renamed from C6; footprint Capacitor_SMD:C_0402_1005Metric_Pad0.74x0.62mm_HandSolder -> Capacitor_SMD:C_0201_0603Metric
- C2: renamed from C5; value 4.7uF -> 10uF; footprint Capacitor_SMD:C_0402_1005Metric_Pad0.74x0.62mm_HandSolder -> Capacitor_SMD:C_0402_1005Metric
- C3: renamed from C2; value 4.7uF -> 10uF; footprint Capacitor_SMD:C_0402_1005Metric_Pad0.74x0.62mm_HandSolder -> Capacitor_SMD:C_0402_1005Metric
- C5: renamed from C3; footprint Capacitor_SMD:C_0402_1005Metric_Pad0.74x0.62mm_HandSolder -> Capacitor_SMD:C_0603_1608Metric
- C6: renamed from C4; footprint Capacitor_SMD:C_0402_1005Metric_Pad0.74x0.62mm_HandSolder -> Capacitor_SMD:C_0201_0603Metric
- C7: renamed from C13; footprint Capacitor_SMD:C_0402_1005Metric_Pad0.74x0.62mm_HandSolder -> Capacitor_SMD:C_0201_0603Metric
- C8: renamed from C7; footprint Capacitor_SMD:C_0402_1005Metric_Pad0.74x0.62mm_HandSolder -> Capacitor_SMD:C_0201_0603Metric
- C9: renamed from C8; footprint Capacitor_SMD:C_0402_1005Metric_Pad0.74x0.62mm_HandSolder -> Capacitor_SMD:C_0201_0603Metric
- D1: value LED -> RED; footprint LED_SMD:LED_0402_1005Metric_Pad0.77x0.64mm_HandSolder -> LED_SMD:LED_0402_1005Metric
- D2: footprint LED_SMD:LED_0402_1005Metric_Pad0.77x0.64mm_HandSolder -> LED_SMD:LED_0402_1005Metric
- P1: footprint Connector_USB:USB_C_Receptacle_XKB_U262-16XN-4BVC11 -> Connector_USB:USB_C_Receptacle_GCT_USB4105-xx-A_16P_TopMnt_Horizontal
- R1: renamed from R3; footprint Resistor_SMD:R_0402_1005Metric_Pad0.72x0.64mm_HandSolder -> Resistor_SMD:R_0201_0603Metric
- R10: renamed from R2; value 1K -> 2K; footprint Resistor_SMD:R_0402_1005Metric_Pad0.72x0.64mm_HandSolder -> Resistor_SMD:R_0201_0603Metric
- R14: renamed from R5; footprint Resistor_SMD:R_0402_1005Metric_Pad0.72x0.64mm_HandSolder -> Resistor_SMD:R_0201_0603Metric
- R15: renamed from R4; footprint Resistor_SMD:R_0402_1005Metric_Pad0.72x0.64mm_HandSolder -> Resistor_SMD:R_0201_0603Metric
- R2: renamed from R1; value 1K -> 4.7K; footprint Resistor_SMD:R_0402_1005Metric_Pad0.72x0.64mm_HandSolder -> Resistor_SMD:R_0201_0603Metric
- R6: value 10K -> 2K; footprint Resistor_SMD:R_0402_1005Metric_Pad0.72x0.64mm_HandSolder -> Resistor_SMD:R_0402_1005Metric
- R7: value 10K -> 3K3; footprint Resistor_SMD:R_0402_1005Metric_Pad0.72x0.64mm_HandSolder -> Resistor_SMD:R_0201_0603Metric
- R8: value 10K -> 2K; footprint Resistor_SMD:R_0402_1005Metric_Pad0.72x0.64mm_HandSolder -> Resistor_SMD:R_0201_0603Metric
- R9: value 1K -> 0.8R; footprint Resistor_SMD:R_0402_1005Metric_Pad0.72x0.64mm_HandSolder -> Resistor_SMD:R_0201_0603Metric
- renumbered U5 to U4
Connections:
- net CHIP_PU is gone; now on an unnamed net: R6.2
- net DTR is gone; now on net VBUS: R7.1
- net LED is gone; now on net VBUS: R9.1
- net RTS is gone; now on net SP_USB: R8.1
- net +3V3: now also D3.4 (VDD), R11.1, R12.1, R13.1, U2.13 (VDD), U2.8 (VLOGIC), U3.3 (3V3); no longer R6.1
- net +BATT: now also R3.1, TP2.1, U1.3 (BAT)
- net GND: now also R6.1, R8.2, C4.2, D3.2 (VSS), R4.2, R5.1, SW1.2 (B), SW2.2 (B), TP1.1, U1.2 (GND), U2.18 (GND), U3.1 (GND), U3.11 (GND), U3.14 (GND), U3.2 (GND), U3.36 (GND), U3.37 (GND), U3.38 (GND), U3.39 (GND), U3.40 (GND), U3.41 (GND), U3.42 (GND), U3.43 (GND), U3.44 (GND), U3.45 (GND), U3.46 (GND), U3.47 (GND), U3.48 (GND), U3.49 (GND), U3.50 (GND), U3.51 (GND), U3.52 (GND), U3.53 (GND)
- net RGB_DI: now also D3.3 (DIN), U3.16 (GPIO10)
- net SCL: now also U2.23 (SCL), U3.20 (GPIO6)
- net SDA: now also U2.24 (SDA), U3.19 (GPIO5/ADC2_CH0)
- net VBUS: now also R10.2; no longer R10.1
- net at C5.2: now also U2.10 (REGOUT)
- net at C6.1: now also U2.20 (CPOUT)
- net at R1.1: now also U1.6 (PROG)
- net SP_USB: now reaches R7.2
- net SP_USB: now also U3.6 (GPIO3/ADC1_CH3)
- net at D2.1 (K): now also U1.1 (~{CHRG})
- net at D2.2 (A): now also R10.1; no longer R10.2
- net at R9.2: now also U1.4 (V_{CC})
- net USB_P: now reaches P1.A6 (D+)
- net USB_P: now also U3.27 (GPIO19/USB_D+)
- net USB_N: now reaches P1.A7 (D-)
- net USB_N: now also U3.26 (GPIO18/USB_D-)
- net at P1.B5 (CC2): now also R5.2
- new net: R13.2, U3.22 (GPIO8)
- new net: R12.2, U3.5 (GPIO2/ADC1_CH2)
- new net BOOT: SW1.1 (A), U3.23 (GPIO9)
- new net RESET: C4.1, R11.2, SW2.1 (A), U3.8 (EN/CHIP_PU)
- new net SP_BAT: R3.2, R4.1, U3.18 (GPIO4/ADC1_CH4)
- no-connect marks 40 -> 14
Other:
- moved on the sheet: C1, C2, C3, C5, C6, C7, C8, C9, D4, J2, P1, Q1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

Commit message: Update Board
Parts:
- removed P1: USB_C_Plug_USB2.0, Connector_USB:USB_C_Receptacle_GCT_USB4105-xx-A_16P_TopMnt_Horizontal, symbol Connector:USB_C_Plug_USB2.0
- removed R12, R13: 100K, Resistor_SMD:R_0201_0603Metric, symbol Device:R
- added J1: USB_C_Receptacle_USB2.0_16P, Connector_USB:USB_C_Receptacle_GCT_USB4105-xx-A_16P_TopMnt_Horizontal, symbol Connector:USB_C_Receptacle_USB2.0_16P
- C2, C3: footprint Capacitor_SMD:C_0402_1005Metric -> Capacitor_SMD:C_0201_0603Metric
- R11, R15: value 100K -> 10K
- R5, R6: value 2K -> 5.1K
- SW1, SW2: footprint Button_Switch_SMD:SW_SPST_CK_KMS2xxGP -> Button_Switch_SMD:SW_SPST_B3U-1000P
Connections:
- net GND: now also J1.A1 (GND), J1.A12 (GND), J1.B1 (GND), J1.B12 (GND)
- net USB_N: now also J1.A7 (D-), J1.B7 (D-)
- net USB_P: now also J1.A6 (D+), J1.B6 (D+)
- net VBUS: now also J1.A4 (VBUS), J1.A9 (VBUS), J1.B4 (VBUS), J1.B9 (VBUS)
- net at R5.2: now also J1.B5 (CC2)
- net at R6.2: now also J1.A5 (CC1)
- no-connect marks 14 -> 18
Other:
- moved on the sheet: R5, R6

Commit message: Update Board
Parts:
- removed D4: SS34, Diode_SMD:D_SMA, symbol Diode:SS34
- removed J2: Sh 1.0, Connector_JST:JST_SH_SM04B-SRSS-TB_1x04-1MP_P1.00mm_Horizontal, symbol Connector_Generic:Conn_01x04
- removed R7: 3K3, Resistor_SMD:R_0201_0603Metric, symbol Device:R
- removed R8: 2K, Resistor_SMD:R_0201_0603Metric, symbol Device:R
- removed R9: 0.8R, Resistor_SMD:R_0201_0603Metric, symbol Device:R
- removed TP1, TP2: TestPoint, TestPoint:TestPoint_Pad_D1.5mm, symbol Connector:TestPoint
- added D4: MBR0530, Diode_SMD:D_SOD-123, symbol Diode:MBR0530
- added J1: PH2.0, Connector_JST:JST_PH_B2B-PH-SM4-TB_1x02-1MP_P2.00mm_Vertical, symbol Connector_Generic_MountingPin:Conn_01x02_MountingPin
- added J3: SH1.0, Connector_JST:JST_SH_BM04B-SRSS-TB_1x04-1MP_P1.00mm_Vertical, symbol Connector_Generic_MountingPin:Conn_01x04_MountingPin
- added R1: 10K, Resistor_SMD:R_0402_1005Metric, symbol Device:R
- added SW3: SW_SPDT_312, Button_Switch_SMD:SW_SPDT_PCM12, symbol Switch:SW_SPDT_312
- C1, C2, C3, C7, C8, C9: footprint Capacitor_SMD:C_0201_0603Metric -> Capacitor_SMD:C_0402_1005Metric
- C4, C6: value 0.1uF -> 100nF; footprint Capacitor_SMD:C_0201_0603Metric -> Capacitor_SMD:C_0402_1005Metric
- D2: value LED -> BLUE
- J2: renamed from J1; footprint Connector_USB:USB_C_Receptacle_GCT_USB4105-xx-A_16P_TopMnt_Horizontal -> Connector_USB:USB_C_Receptacle_GCT_USB4110
- R10, R11: footprint Resistor_SMD:R_0201_0603Metric -> Resistor_SMD:R_0402_1005Metric
- R12: renamed from R14; footprint Resistor_SMD:R_0201_0603Metric -> Resistor_SMD:R_0402_1005Metric
- R13: renamed from R15; footprint Resistor_SMD:R_0201_0603Metric -> Resistor_SMD:R_0402_1005Metric
- R2: renamed from R1; footprint Resistor_SMD:R_0201_0603Metric -> Resistor_SMD:R_0402_1005Metric
- R3: renamed from R2; value 4.7K -> 2K; footprint Resistor_SMD:R_0201_0603Metric -> Resistor_SMD:R_0402_1005Metric
- SW1, SW2: footprint Button_Switch_SMD:SW_SPST_B3U-1000P -> Button_Switch_SMD:SW_Push_SPST_NO_Alps_SKRK
- renumbered R3 to R4, R4 to R5, R5 to R6, R6 to R7
Connections:
- net +3V3: now also J3.4 (Pin_4), SW3.1 (B); no longer C8.1, C9.1, U4.5 (VOUT)
- net +BATT: now also J1.1 (Pin_1)
- net BOOT: now also R1.1; no longer SW1.1 (A)
- net GND: now also J1.2 (Pin_2), J1.MP (MountPin), J3.3 (Pin_3), J3.MP (MountPin)
- net SCL: now also J3.1 (Pin_1)
- net SDA: now also J3.2 (Pin_2)
- net VBUS: now also U1.4 (V_{CC}), D4.2 (A)
- net at C7.1, Q1.2 (S), R13.1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: now also D4.1 (K)
- new net: C8.1, C9.1, SW3.2 (C), U4.5 (VOUT)
- new net: R1.2, SW1.1 (A)
- no-connect marks 18 -> 19

Commit message: Update Board
Parts:
- U2: footprint Sensor_Motion:InvenSense_QFN-24_4x4mm_P0.5mm_NoMask -> Sensor_Motion:InvenSense_QFN-24_4x4mm_P0.5mm
Connections:
- net +3V3: now also J3.3 (Pin_3); no longer J3.4 (Pin_4)
- net +BATT: now also J1.2 (Pin_2); no longer J1.1 (Pin_1)
- net GND: now also J1.1 (Pin_1), J3.4 (Pin_4); no longer J1.2 (Pin_2), J3.3 (Pin_3)
- net SP_USB: no longer names the net of U3.6 (GPIO3/ADC1_CH3)
- no-connect marks 19 -> 20
Other:
- moved on the sheet: J1

Commit message: Update Board
Parts:
- removed C5: 2.2nF, Capacitor_SMD:C_0603_1608Metric, symbol Device:C
- removed C6: 100nF, Capacitor_SMD:C_0402_1005Metric, symbol Device:C
- removed U2: MPU-6050, Sensor_Motion:InvenSense_QFN-24_4x4mm_P0.5mm, symbol Sensor_Motion:MPU-6050
- added C10, C11, C12: 1uF, Capacitor_SMD:C_0402_1005Metric, symbol Device:C
- added C13: 0.1uF, Capacitor_SMD:C_0402_1005Metric, symbol Device:C
- added R14, R9: 10K, Resistor_SMD:R_0402_1005Metric, symbol Device:R
- added R15, R8: NC, Resistor_SMD:R_0402_1005Metric, symbol Device:R
- added U5: XC6206P182MR, Package_TO_SOT_SMD:SOT-23-3, symbol Regulator_Linear:XC6206PxxxMR
- added U6: MPU-9250, Sensor_Motion:InvenSense_QFN-24_3x3mm_P0.4mm, symbol Sensor_Motion:MPU-9250
Connections:
- net +3V3: now also C10.1, R14.2, R8.2, R9.1, U5.3 (VI)
- net GND: now also C10.2, C11.2, C12.2, C13.2, R15.2, U5.1 (GND), U6.18 (GND), U6.20 (RESV_GND)
- net SCL: now also R14.1, U6.23 (SCL/SCLK)
- net SDA: now also R9.2, U6.24 (SDA/MOSI)
- new net: R15.1, U6.1 (RESV_VDDIO)
- new net: C13.1, U6.10 (REGOUT)
- new net +1V8: C11.1, C12.1, R8.1, U5.2 (VO), U6.13 (VDD), U6.8 (VDDIO)
