File: C3-1.kicad_pcb (KiCad board)
At the start: 2 copper layers, 23.2 x 21.3 mm, 36 parts, among them J1 PH2.0, J2 USB_C_Receptacle_USB2.0_16P, J3 SH1.0, Q1 AO3401A, SW1 Boot, SW2 Reset, SW3 SW_SPDT_312, U1 TP4057, U2 MPU-6050, U3 ESP32-C3-MINI-1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

Commit message: Update Board
Parts:
- moved R11 110.8 mm to (121.2, 51.8), turned to 180 degrees
- moved C4 109.8 mm to (119.7, 52.3), turned to -90 degrees
- moved C1 108.8 mm to (121.7, 53.4), turned to -90 degrees
- moved SW2 108.6 mm to (123.9, 54.1), turned to -90 degrees
- moved C5 107.1 mm to (118.9, 54.0), turned to 180 degrees
- moved U2 105.2 mm to (114.2, 54.7), turned to 0 degrees
- moved R5 104.6 mm to (119.2, 55.9), turned to 0 degrees
- moved U3 103.7 mm to (124.0, 57.7), turned to -90 degrees
- moved U4 101.9 mm to (124.3, 59.1), turned to 90 degrees
- moved D3 101.0 mm to (113.7, 57.6), turned to 0 degrees
- moved C6 100.9 mm to (116.7, 58.1), turned to 0 degrees
- moved R12 99.7 mm to (118.0, 59.2), turned to 0 degrees
- moved R4 98.9 mm to (120.2, 60.3), turned to 90 degrees
- moved R13 98.7 mm to (121.9, 60.8), turned to 90 degrees
- moved R1 98.6 mm to (113.3, 59.2), turned to 180 degrees
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Routing:
- net SP_BAT: track 8.21 -> 8.85 mm
- net GND: track 50.0 -> 50.1 mm, vias 18 -> 19
Other:
- board size 23.2 x 21.3 mm -> 21.4 x 23.1 mm
- board text added: "C3-1"

Commit message: Update Board
Routing:
- net GND: track 50.1 -> 60.6 mm
- net +3V3: track 69.6 -> 70.2 mm
Other:
- board size 21.4 x 23.1 mm -> 21.9 x 23.1 mm
