File: AIO.kicad_pcb (KiCad board)
At the start: 2 copper layers, 91 x 78 mm, 359 parts, among them J1 Conn_01x02_MountingPin, J1 JST SH1.0, J1 PH2.0, J1 SH1.0, J1 Sh 1.0, J2 SH1.0, J2 USB_C_Receptacle_PowerOnly_6P, J2 USB_C_Receptacle_USB2.0_16P, J3 JST PH2.0, J3 SH1.0, J3 USB_C_Receptacle_PowerOnly_6P, J3 USB_C_Receptacle_USB2.0_16P, Q1 AO3401A, Q2 AO3400A, Q2 MBT3904DW1, SW1 Boot, SW1 Reset, SW1 SW_Push, SW1 SW_SPDT, SW2 Boot, SW2 Reset, SW2 SW_Push, SW2 SW_SPDT, SW3 Boot, SW3 SW_Push_SPDT, SW3 SW_SPDT, SW3 SW_SPDT_312, U1 AP2112K-3.3, U1 MPU-6050, U1 TP4057, U1 XC6206P182MR, U2 AP2112K-3.3, U2 ESP32-S3-WROOM-1, U2 ESP32-WROOM-32U, U2 IP5306, U2 MPU-6050, U3 ESP32-C3-MINI-1, U3 ESP32C3_SuperMini, U3 MCP73831-2-OT, U3 ME6211C33M5, U3 MPU-9250, U4 AP2112K-3.3, U4 MCP73831-2-OT, U4 MPU-6050, U4 TP4057, U5 ESP32-S2, U5 XC6206P182MR, U6 MPU-9250, Y1 40MHz

Commit message: Update Board
Parts:
- C1: footprint Capacitor_SMD:C_0201_0603Metric -> Capacitor_SMD:C_0402_1005Metric
- R2, R4: footprint Resistor_SMD:R_0201_0603Metric -> Resistor_SMD:R_0402_1005Metric
- moved R2 0.47 mm to (218.2, 75.0)
- moved R4 0.29 mm to (224.2, 69.8)
- moved C4 0.16 mm to (209.7, 74.7)
- moved C1 0.16 mm to (229.8, 78.9)
- moved C10 0.16 mm to (217.0, 81.9)
- moved C11 0.16 mm to (226.7, 80.2)
- moved C12 0.16 mm to (226.7, 81.2)
- moved C13 0.16 mm to (217.0, 80.8)
- moved C14 0.16 mm to (215.1, 79.9)
- moved C2 0.16 mm to (228.8, 65.8)
- moved C5 0.16 mm to (213.0, 74.6)
- moved C6 0.16 mm to (217.5, 77.1)
- moved C7 0.16 mm to (216.3, 77.9)
- moved C8 0.16 mm to (226.7, 82.3)
- moved C9 0.16 mm to (217.1, 83.0)
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Connections:
- J2 pad S1: unconnected-(J2-SHIELD-PadS1)_3 -> unconnected-(J2-SHIELD-PadS1)_1
Routing:
- net GND: track 359.0 -> 357.5 mm
- net VBUS: track 220.4 -> 221.3 mm
- net Net-(D3-A): track 14.9 -> 15.6 mm
- net Net-(R4-Pad1): track 12.6 -> 13.1 mm
