File: mC3.kicad_pcb (KiCad board)
At the start: 2 copper layers, 19.7 x 31.4 mm, 36 parts, among them J1 Sh 1.0, J2 USB_C_Receptacle_PowerOnly_6P, Q1 AO3401A, SW1 SW_Push, SW2 SW_SPDT, U1 MPU-6050, U2 IP5306, U3 ESP32C3_SuperMini

Commit message: Update Board
Routing:
- net GND: vias 23 -> 24
Changed lines of the file:
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@@
 		(tags "capacitor")
 		(property "Reference" "C6"
-			(at 0 -1.16 360)
+			(at 0 -1.16 0)
 			(layer "F.SilkS")
 			(hide yes)
@@
 		)
 		(property "Value" "10uF"
-			(at 0 1.16 360)
+			(at 0 1.16 0)
 			(layer "F.Fab")
 			(hide yes)
@@
 		)
 		(fp_text user "${REFERENCE}"
-			(at 0 0 360)
+			(at 0 0 0)
 			(layer "F.Fab")
 			(effects
@@
 		(tags "test point SMD pad")
 		(property "Reference" "TP1"
-			(at 0 -1.648 360)
+			(at 0 -1.648 0)
 			(layer "F.SilkS")
 			(hide yes)
@@
 		)
 		(property "Value" "Bat+"
-			(at 0 1.75 360)
+			(at 0 1.75 0)
 			(layer "F.Fab")
 			(hide yes)
@@
 		(tags "capacitor")
 		(property "Reference" "C5"
-			(at 0 -1.16 360)
+			(at 0 -1.16 0)
 			(layer "F.SilkS")
 			(hide yes)
@@
 		)
 		(property "Value" "0.1uF"
-			(at 0 1.16 360)
+			(at 0 1.16 0)
 			(layer "F.Fab")
 			(hide yes)
@@
 		)
 		(fp_text user "${REFERENCE}"
-			(at 0 0 360)
+			(at 0 0 0)
 			(layer "F.Fab")
 			(effects
@@
 		(tags "LED")
 		(property "Reference" "D4"
-			(at 0 -1.17 360)
+			(at 0 -1.17 0)
 			(layer "F.SilkS")
 			(hide yes)
@@
 		)
 		(property "Value" "LED"
-			(at 0 1.17 360)
+			(at 0 1.17 0)
 			(layer "F.Fab")
 			(hide yes)
@@
 		)
 		(fp_text user "${REFERENCE}"
-			(at 0 0 360)
+			(at 0 0 0)
 			(layer "F.Fab")
 			(effects
@@
 		(tags "LED")
 		(property "Reference" "D3"
-			(at 0 -1.17 360)
+			(at 0 -1.17 0)
 			(layer "F.SilkS")
 			(hide yes)
@@
 		)
 		(property "Value" "LED"
-			(at 0 1.17 360)
+			(at 0 1.17 0)
 			(layer "F.Fab")
 			(hide yes)
@@
 		)
 		(fp_text user "${REFERENCE}"
-			(at 0 0 360)
+			(at 0 0 0)
 			(layer "F.Fab")
 			(effects
@@
 		(tags "resistor")
 		(property "Reference" "R3"
-			(at 0 -1.17 360)
+			(at 0 -1.17 0)
 			(layer "F.SilkS")
 			(hide yes)
@@
 		)
 		(property "Value" "2R"
-			(at 0 1.17 360)
+			(at 0 1.17 0)
 			(layer "F.Fab")
 			(hide yes)
@@
 		)
 		(fp_text user "${REFERENCE}"
-			(at 0 0 360)
+			(at 0 0 0)
 			(layer "F.Fab")
 			(effects
@@
 		(tags "capacitor")
 		(property "Reference" "C3"
-			(at 0 -1.16 360)
+			(at 0 -1.16 0)
 			(layer "F.SilkS")
 			(hide yes)
@@
 		)
 		(property "Value" "10uF"
-			(at 0 1.16 360)
+			(at 0 1.16 0)
 			(layer "F.Fab")
 			(hide yes)
@@
 		)
 		(fp_text user "${REFERENCE}"
-			(at 0 0 360)
+			(at 0 0 0)
 			(layer "F.Fab")
 			(effects
@@
 		(at 105.565 35.2825)
 		(property "Reference" "U2"
-			(at -3.429 -0.635 360)
+			(at -3.429 -0.635 0)
 			(layer "F.SilkS")
 			(hide yes)
@@
 		)
 		(property "Value" "IP5306"
-			(at 3.175 -1.143 360)
+			(at 3.175 -1.143 0)
 			(layer "F.Fab")
 			(hide yes)
@@
 		)
 		(property "Footprint" "Custom:IP5306"
-			(at 0 0 360)
+			(at 0 0 0)
 			(layer "F.Fab")
 			(hide yes)
@@
 		)
 		(property "Datasheet" ""
-			(at 0 0 360)
+			(at 0 0 0)
 			(layer "F.Fab")
 			(hide yes)
@@
 		)
 		(property "Description" ""
-			(at 0 0 360)
+			(at 0 0 0)
 			(layer "F.Fab")
 			(hide yes)
@@
 		(tags "resistor")
 		(property "Reference" "R2"
-			(at 0 -1.05 360)
+			(at 0 -1.05 0)
 			(layer "F.SilkS")
 			(hide yes)
@@
 		)
 		(property "Value" "10K"
-			(at 0 1.05 360)
+			(at 0 1.05 0)
 			(layer "F.Fab")
 			(hide yes)
@@
 		)
 		(fp_text user "${REFERENCE}"
-			(at 0 -0.68 360)
+			(at 0 -0.68 0)
 			(layer "F.Fab")
 			(effects
@@
 		(tags "LED")
 		(property "Reference" "D5"
-			(at 0 -1.17 360)
+			(at 0 -1.17 0)
 			(layer "F.SilkS")
 			(hide yes)
@@
 		)
 		(property "Value" "LED"
-			(at 0 1.17 360)
+			(at 0 1.17 0)
 			(layer "F.Fab")
 			(hide yes)
@@
 		)
 		(fp_text user "${REFERENCE}"
-			(at 0 0 360)
+			(at 0 0 0)
 			(layer "F.Fab")
 			(effects
@@
 		(tags "QFN 0.5")
 		(property "Reference" "U1"
-			(at 0 -3.375 360)
+			(at 0 -3.375 0)
 			(layer "F.SilkS")
 			(hide yes)
@@
 		)
 		(property "Value" "MPU-6050"
-			(at 0 3.375 360)
+			(at 0 3.375 0)
 			(layer "F.Fab")
 			(hide yes)
@@
 		)
 		(fp_text user "Component"
-			(at 0 0.55 360)
+			(at 0 0.55 0)
 			(layer "Cmts.User")
 			(effects
@@
 		)
 		(fp_text user "KEEPOUT"
-			(at 0 -0.5 360)
+			(at 0 -0.5 0)
 			(layer "Cmts.User")
 			(effects
@@
 		)
 		(fp_text user "No Copper"
-			(at 0 -0.1 360)
+			(at 0 -0.1 0)
 			(layer "Cmts.User")
 			(effects
@@
 		)
 		(fp_text user "Directly Below"
-			(at 0 0.25 360)
+			(at 0 0.25 0)
 			(layer "Cmts.User")
 			(effects
@@
 		)
 		(fp_text user "${REFERENCE}"
-			(at 0 0 360)
+			(at 0 0 0)
 			(layer "F.Fab")
 			(effects
@@
 		(tags "Diode SMA (DO-214AC)")
 		(property "Reference" "D2"
-			(at 0 -2.5 360)
+			(at 0 -2.5 0)
 			(layer "F.SilkS")
 			(hide yes)
@@
 		)
 		(property "Value" "SS54"
-			(at 0 2.6 360)
+			(at 0 2.6 0)
 			(layer "F.Fab")
 			(hide yes)
@@
 		(tags "test point SMD pad")
 		(property "Reference" "TP2"
-			(at 0 -1.648 360)
+			(at 0 -1.648 0)
 			(layer "F.SilkS")
 			(hide yes)
@@
 		)
 		(property "Value" "Bat-"
-			(at 0 1.75 360)
+			(at 0 1.75 0)
 			(layer "F.Fab")
 			(hide yes)
@@
 		(tags "Choke SMD")
 		(property "Reference" "L1"
-			(at 0 -4.45 360)
+			(at 0 -4.45 0)
 			(layer "F.SilkS")
 			(hide yes)
@@
 		)
 		(property "Value" "1R0"
-			(at 0 4.45 360)
+			(at 0 4.45 0)
 			(layer "F.Fab")
 			(hide yes)
@@
 		)
 		(fp_text user "${REFERENCE}"
-			(at 0 0 360)
+			(at 0 0 0)
 			(layer "F.Fab")
 			(effects
@@
 		(tags "resistor")
 		(property "Reference" "R5"
-			(at 0 -1.17 360)
+			(at 0 -1.17 0)
 			(layer "F.SilkS")
 			(hide yes)
@@
 		)
 		(property "Value" "2R"
-			(at 0 1.17 360)
+			(at 0 1.17 0)
 			(layer "F.Fab")
 			(hide yes)
@@
 		)
 		(fp_text user "${REFERENCE}"
-			(at 0 0 360)
+			(at 0 0 0)
 			(layer "F.Fab")
 			(effects
@@
 		(tags "LED")
 		(property "Reference" "D6"
-			(at 0 -1.17 360)
+			(at 0 -1.17 0)
 			(layer "F.SilkS")
 			(hide yes)
@@
 		)
 		(property "Value" "LED"
-			(at 0 1.17 360)
+			(at 0 1.17 0)
 			(layer "F.Fab")
 			(hide yes)
@@
 		)
 		(fp_text user "${REFERENCE}"
-			(at 0 0 360)
+			(at 0 0 0)
 			(layer "F.Fab")
 			(effects
@@
 		(tags "capacitor")
 		(property "Reference" "C7"
-			(at 0 -1.16 360)
+			(at 0 -1.16 0)
 			(layer "F.SilkS")
 			(hide yes)
@@
 		)
 		(property "Value" "10uF"
-			(at 0 1.16 360)
+			(at 0 1.16 0)
 			(layer "F.Fab")
 			(hide yes)
@@
 		)
 		(fp_text user "${REFERENCE}"
-			(at 0 0 360)
+			(at 0 0 0)
 			(layer "F.Fab")
 			(effects
@@
 		(tags "capacitor")
 		(property "Reference" "C14"
-			(at 0 -1.16 360)
+			(at 0 -1.16 0)
 			(layer "F.SilkS")
 			(hide yes)
@@
 		)
 		(property "Value" "1.0uF"
-			(at 0 1.16 360)
+			(at 0 1.16 0)
 			(layer "F.Fab")
 			(hide yes)
@@
 		)
 		(fp_text user "${REFERENCE}"
-			(at 0 0 360)
+			(at 0 0 0)
 			(layer "F.Fab")
 			(effects
@@
 		(tags "capacitor")
 		(property "Reference" "C1"
-			(at 0 -1.05 360)
+			(at 0 -1.05 0)
 			(layer "F.SilkS")
 			(hide yes)
@@
 		)
 		(property "Value" "1.0uF"
-			(at 0 1.05 360)
+			(at 0 1.05 0)
 			(layer "F.Fab")
 			(hide yes)
@@
 		)
 		(fp_text user "${REFERENCE}"
-			(at 0 -0.68 360)
+			(at 0 -0.68 0)
 			(layer "F.Fab")
 			(effects
@@
 		(at 103.7375 40.9725 180)
 		(property "Reference" "U3"
-			(at -5.715 13.6525 360)
+			(at -5.715 13.6525 0)
 			(layer "B.SilkS")
 			(hide yes)
@@
 		)
 		(property "Value" "ESP32C3_SuperMini"
-			(at 6.985 -12.3825 360)
+			(at 6.985 -12.3825 0)
 			(layer "B.Fab")
 			(hide yes)
@@
 		)
 		(property "Footprint" "Custom:ESP32C3_Supermini_SMD"
-			(at 0 0 360)
+			(at 0 0 0)
 			(layer "B.Fab")
 			(hide yes)
@@
 		)
 		(property "Datasheet" ""
-			(at 0 0 360)
+			(at 0 0 0)
 			(layer "B.Fab")
 			(hide yes)
@@
 		)
 		(property "Description" ""
-			(at 0 0 360)
+			(at 0 0 0)
 			(layer "B.Fab")
 			(hide yes)
@@
 	)
 	(via
-		(at 109.71 32.76)
+		(at 109.56494 32.839924)
 		(size 0.6)
 		(drill 0.3)
@@
 		(net 2)
 	)
+	(via
+		(at 109.29 27.74)
+		(size 0.6)
+		(drill 0.3)
+		(layers "F.Cu" "B.Cu")
+		(free yes)
+		(net 2)
+	)

Commit message: Update mC3.kicad_pcb
Parts:
- C1, C10, C11, C12, C13, C14, C2, C3, C4, C5, C6, C7, C8, C9, D2, D3, D4, D5, D6, G***, J1, J2, L1, Q1, R2, R3, R4, R5, SW2, TP1, TP2, U1, U2: moved to B.Cu
- D7, SW1, U3: moved to F.Cu
- moved C9 19.9 mm to (115.5, 40.9)
- moved G*** 19.0 mm to (115.1, 46.6), turned to 0 degrees
- moved SW2 19.0 mm to (115.0, 25.7)
- moved C8 18.5 mm to (114.8, 31.3)
- moved C10 17.6 mm to (114.4, 40.9)
- moved C12 16.3 mm to (113.7, 31.3)
- moved C13 15.4 mm to (113.3, 40.9)
- moved C2 14.6 mm to (98.3, 29.2)
- moved C11 14.2 mm to (112.6, 31.3)
- moved C14 13.7 mm to (112.4, 42.9), turned to 180 degrees
- moved L1 13.3 mm to (112.2, 36.4), turned to 180 degrees
- moved D4 13.2 mm to (99.0, 35.8), turned to 180 degrees
- moved D5 13.2 mm to (99.0, 37.0), turned to 0 degrees
- moved D6 13.2 mm to (99.0, 38.3), turned to 180 degrees
- moved D3 13.2 mm to (99.0, 34.6), turned to 0 degrees
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Other:
- board size 19.7 x 31.4 mm -> 19.7 x 30.7 mm

Commit message: Update Board
Parts:
- C1: footprint Capacitor_SMD:C_0201_0603Metric -> Capacitor_SMD:C_0402_1005Metric
- R2, R4: footprint Resistor_SMD:R_0201_0603Metric -> Resistor_SMD:R_0402_1005Metric
- moved R4 0.43 mm to (102.2, 33.7)
- moved R2 0.39 mm to (107.4, 39.7)
Routing:
- net GND: track 15.2 -> 13.7 mm
- net VBUS: track 32.1 -> 33.0 mm
- net Net-(D3-A): track 11.5 -> 12.2 mm
- net Net-(R4-Pad1): track 12.6 -> 13.1 mm
